File: hardware/esp32-multisensor-pcb.kicad_sch (KiCad schematic)
At the start: 0 parts

Commit message: Complete USB connector schematic connections
Parts:
- added C1: 0.1uF, symbol Device:C_Small
- added D1, D2, D3: LED, symbol Device:LED_Small_Filled
- added F1: 0ZCH0110AF2E, FUSC3226X100N, symbol 0ZCH0110AF2E:0ZCH0110AF2E
- added J1: SS-52400-002, SS-52400-002:BELFUSE_SS-52400-002, symbol SS-52400-002:SS-52400-002
- added J2: B2B-PH-SM4-TB, B2B-PH-SM4-TB:JST_B2B-PH-SM4-TB, symbol B2B-PH-SM4-TB:B2B-PH-SM4-TB
- added R1, R2: 10k, symbol Device:R_Small_US
- added R3, R4: 5k1, symbol Device:R_Small_US
- added R5: 2k, symbol Device:R_Small_US
- added R6: 20k, symbol Device:R_Small_US
- added R7, R8, R9: 470, symbol Device:R_Small_US
- added U2: MCP73871, Package_DFN_QFN:QFN-20-1EP_4x4mm_P0.5mm_EP2.5x2.5mm, symbol Battery_Management:MCP73871
- added VR1: LM1117MPX-3.3, LM1117MPX-3.3:VREG_LM1117MPX-3.3, symbol LM1117MPX-3.3:LM1117MPX-3.3
Connections:
- new net: J1.A5 (CC1), R4.1
- new net: J1.B5 (CC2), R3.1
- new net: D2.1 (K), R8.1
- new net: R8.2, U2.8 (STAT1/~{LBO})
- new net: R2.2, U2.5 (THERM)
- new net: R5.2, U2.13 (PROG1)
- new net: D3.1 (K), R9.1
- new net: U2.1 (OUT), U2.20 (OUT)
- new net: U2.10 (V_{SS}), U2.11 (V_{SS}), U2.21 (V_{SS})
- new net: R6.2, U2.12 (PROG3)
- new net: U2.14 (V_{BAT}), U2.15 (V_{BAT})
- new net: U2.18 (IN), U2.19 (IN)
- new net: R9.2, U2.6 (~{PG})
- new net: R7.2, U2.7 (STAT2)
- new net: R1.2, U2.9 (~{TE})
- new net: D1.1 (K), R7.1
- new net +5V_USB: F1.2
- new net GND: C1.2, J1.A1 (GNDA1), J1.A12 (GNDA2), J1.B1 (GNDB1), J1.B12 (GNDB2), J1.G1 (GND/SHIELD), J1.G2 (GND/SHIELD), J1.G3 (GND/SHIELD), J1.G4 (GND/SHIELD), J1.S1 (GND/SHIELD), J1.S2 (GND/SHIELD), J1.S3 (GND/SHIELD), J1.S4 (GND/SHIELD), R1.1, R2.1, R3.2, R4.2, R5.1, R6.1
- new net USB_DN: J1.A7 (DN1), J1.B7 (DN2)
- new net USB_DP: J1.A6 (DP1), J1.B6 (DP2)
- new net VBUS: C1.1, F1.1, J1.A4 (VBUSA1), J1.B4 (VBUSB1), J1.B9 (VBUSB2)
- no-connect marks 0 -> 10
