File: hardware/esp32-c3-02.kicad_sch (KiCad schematic)
At the start: 15 parts, among them J3 microSD, U1 ESP32-C3-WROOM-02-H4, U3 CP2102N-Axx-xQFN20, U4 USBLC6-2SC6, U5 W25Q32JVSSIQ

Commit message: feat: add ESP32 C3 module connections
Parts:
- added C10: 10uF, symbol Device:C_Polarized_Small_US
- added C11: 0.1uF, symbol Device:C_Small
- added R16, R17: 50, symbol Device:R_Small_US
Connections:
- net UART_RX is gone; now on net ESP32_RX: U3.17 (RXD)
- net UART_TX is gone; now on net ESP32_TX: U3.18 (TXD)
- net +3.3V: now also U1.1 (3V3), C10.1, C11.1
- net GND: now also U1.19 (GND), U1.20 (GND), U1.21 (GND), U1.22 (GND), U1.23 (GND), U1.24 (GND), U1.25 (GND), U1.26 (GND), U1.27 (GND), U1.28 (GND), U1.29 (GND), U1.30 (GND), U1.31 (GND), U1.32 (GND), U1.33 (GND), U1.34 (GND), U1.35 (GND), U1.36 (GND), U1.37 (GND), U1.38 (GND), U1.39 (GND), U1.9 (GND), C10.2, C11.2
- net ESP32_CS: now reaches U1.10 (IO10)
- net ESP32_TX: now reaches U1.11 (RXD)
- net ESP32_RX: now reaches U1.12 (TXD)
- net ESP32_GPIO18: now reaches U1.13 (IO18)
- net ESP32_GPIO19: now reaches U1.14 (IO19)
- net ESP32_SCL: now reaches U1.15 (IO3)
- net ESP32_MISO: now reaches U1.16 (IO2)
- net ESP32_PHOTO: now reaches U1.17 (IO1)
- net ESP32_CD: now reaches U1.18 (IO0)
- net ESP32_EN: now reaches U1.2 (EN)
- net ESP32_SDA: now reaches U1.3 (IO4)
- net ESP32_MIC: now reaches U1.4 (IO5)
- net at U1.5 (IO6): now also R16.2
- net at U1.6 (IO7): now also R17.2
- net ESP32_GPIO8: now reaches U1.7 (IO8)
- net ESP32_BOOT: now reaches U1.8 (IO9)
- new net ESP32_MOSI: R17.1
- new net ESP32_SCLK: R16.1
Other:
- note added: "ESP32 C3 module"
- moved on the sheet: C7, J3, R11, R12, U1, U4, U5
