File: hardware/_restore_backup_2026-07-17T14-48-00-328/esp32-multisensor-pcb.kicad_sch (KiCad schematic)
At the start: 19 parts, among them J1 SS-52400-002, J2 B2B-PH-SM4-TB, U2 MCP73871

Commit message: feat: add LiPo battery charger module
Parts:
- removed C2: 0.1uF, symbol Device:C_Small
Connections:
- net +5V_USB: no longer D1.2 (A), D2.2 (A), D3.2 (A), U2.17 (CE), U2.18 (IN), U2.19 (IN), U2.2 (VPCC)
- net GND: no longer U2.10 (V_{SS}), U2.11 (V_{SS}), U2.21 (V_{SS})
- net at U2.14 (V_{BAT}), U2.15 (V_{BAT}): no longer U2.16 (V_{BAT_SENSE})
- net at U2.6 (~{PG}): now also R9.2; no longer R7.2
- net at U2.7 (STAT2): now also R7.2; no longer R9.2
- net +5V: no longer names the net of U2.1 (OUT), U2.20 (OUT)
- new net: U2.10 (V_{SS}), U2.11 (V_{SS}), U2.21 (V_{SS})
- new net: U2.18 (IN), U2.19 (IN)
- no-connect marks 11 -> 10
Other:
- note removed: "LiPo Battery Charger"
- note removed: "USB Connector"
- moved on the sheet: D1, D2, D3, R1, R2, R5, R6, R7, R8, R9, U2
